File: Logitech_Unifying/Logitech_Unifying_Expansion_Card_Retrofit.kicad_sch (KiCad schematic)
At the start: 9 parts, among them P1 USB_C_Plug_USB2.0, U1 AP2112K-3.3

Commit message: v1
Parts:
- removed C1, C2: 10uF, Capacitor_SMD:C_0805_2012Metric, symbol Device:C_Small
- removed U1: AP2112K-3.3, Package_TO_SOT_SMD:SOT-23-5, symbol Regulator_Linear:AP2112K-3.3
Other:
- note removed: "5V to 3.3V 600mA"
